File: PCB/TPS42/TPS42.kicad_pcb (KiCad board)
At the start: 2 copper layers, 138.1 x 89.7 mm, 77 parts, among them J1 PJ-320A, J11 Conn_01x06, J14 FH12-10S-0.5SH, J3 TP Sensor Module, J4 TP Module, J6 OLED, J7 TrackPoint, J8 Battery, J9 TP Sensor Module, SW1 SW_DPST_x2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

Commit message: mcu bridges
Routing:
- net GND: track 0.00 -> 44.1 mm, vias 0 -> 3
- net COL3: track 0.00 -> 28.8 mm, vias 0 -> 1
- net COL4: track 0.00 -> 28.4 mm, vias 0 -> 1
- net COL2: track 0.00 -> 25.5 mm, vias 0 -> 1
- net COL5: track 0.00 -> 24.5 mm, vias 0 -> 1
- net COL1: track 0.00 -> 23.7 mm, vias 0 -> 1
- net TP_CLK: track 0.00 -> 22.1 mm, vias 0 -> 1
- net COL0: track 0.00 -> 18.6 mm, vias 0 -> 1
- net TP_DATA: track 0.00 -> 16.8 mm, vias 0 -> 1
- net ROW3: track 0.00 -> 16.3 mm, vias 0 -> 1
- net SERIAL: track 0.00 -> 16.0 mm, vias 0 -> 1
- net BAT+: track 0.00 -> 15.7 mm, vias 0 -> 1
- net ROW2: track 0.00 -> 15.5 mm, vias 0 -> 1
- net CS: track 0.00 -> 14.8 mm, vias 0 -> 1
- net ROW1: track 0.00 -> 14.5 mm, vias 0 -> 1
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
Commit message: Setting some labels
Other:
- board text added: "1"
- board text added: "2"
- board text added: "3"
- board text added: "4"
- board text added: "CLK"
- board text added: "DAT"
- board text added: "GND"
- board text added: "RST"
- board text added: "VCC"
Changed lines of the file:
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@@
     (property "Sheetname" "")
     (attr through_hole)
-    (fp_text reference "S12" (at 0 3.175 180) (layer "F.SilkS")
+    (fp_text reference "S12" (at 0.01 -2.795 180) (layer "F.SilkS")
       (effects (font (size 1 1) (thickness 0.15)))
     )
@@
       (effects (font (size 1 1) (thickness 0.15)))
     )
-    (fp_text user "${REFERENCE}" (at 0 3.175 180) (layer "B.SilkS")
+    (fp_text user "${REFERENCE}" (at 0.02 -2.775 180) (layer "B.SilkS")
       (effects (font (size 1 1) (thickness 0.15)) (justify mirror))
     )
@@
     (fp_line (start 2 -7.7) (end 1.5 -8.2) (layer "F.SilkS") (width 0.15))
     (fp_line (start -7 -6) (end -7 -7) (layer "F.SilkS") (width 0.15))
-    (fp_line (start -7 7) (end -7 6) (layer "F.SilkS") (width 0.15))
     (fp_line (start 7 -7) (end 7 -6) (layer "F.SilkS") (width 0.15))
     (fp_line (start -7 -5.6) (end -7 -6.2) (layer "F.SilkS") (width 0.15))
     (fp_line (start -7 -1.5) (end -7 -2) (layer "F.SilkS") (width 0.15))
-    (fp_line (start -6 7) (end -7 7) (layer "F.SilkS") (width 0.15))
     (fp_line (start 6 -7) (end 7 -7) (layer "F.SilkS") (width 0.15))
     (fp_line (start 7 6) (end 7 7) (layer "F.SilkS") (width 0.15))
@@
     (fp_arc (start -2 -6.7) (mid -2.146447 -6.346447) (end -2.5 -6.2) (layer "F.Fab") (width 0.15))
     (fp_arc (start -2.5 -2.2) (mid -2.06066 -3.26066) (end -1 -3.7) (layer "F.Fab") (width 0.15))
-    (pad "" np_thru_hole circle locked (at -5.5 0 180) (size 1.7018 1.7018) (drill 1.7018) (layers *.Cu *.Mask))
-    (pad "" np_thru_hole circle locked (at 0 -5.95 180) (size 3 3) (drill 3) (layers *.Cu *.Mask))
-    (pad "" np_thru_hole circle locked (at 5.5 0 180) (size 1.7018 1.7018) (drill 1.7018) (layers *.Cu *.Mask))
-    (pad "" np_thru_hole circle locked (at -5 -3.75 180) (size 3 3) (drill 3) (layers *.Cu *.Mask))
-    (pad "" np_thru_hole circle locked (at 5 -3.75 180) (size 3 3) (drill 3) (layers *.Cu *.Mask))
-    (pad "" np_thru_hole circle locked (at 0 0 180) (size 3.429 3.429) (drill 3.429) (layers *.Cu *.Mask))
-    (pad "1" thru_hole circle locked (at 0 5.9 180) (size 2.032 2.032) (drill 1.27) (layers *.Cu *.Mask)
+    (pad "" np_thru_hole circle (at -5.5 0 180) (size 1.7018 1.7018) (drill 1.7018) (layers *.Cu *.Mask))
+    (pad "" np_thru_hole circle (at 0 -5.95 180) (size 3 3) (drill 3) (layers *.Cu *.Mask))
+    (pad "" np_thru_hole circle (at 5.5 0 180) (size 1.7018 1.7018) (drill 1.7018) (layers *.Cu *.Mask))
+    (pad "" np_thru_hole circle (at -5 -3.75 180) (size 3 3) (drill 3) (layers *.Cu *.Mask))
+    (pad "" np_thru_hole circle (at 5 -3.75 180) (size 3 3) (drill 3) (layers *.Cu *.Mask))
+    (pad "" np_thru_hole circle (at 0 0 180) (size 3.429 3.429) (drill 3.429) (layers *.Cu *.Mask))
+    (pad "1" thru_hole circle (at 0 5.9 180) (size 2.032 2.032) (drill 1.27) (layers *.Cu *.Mask)
       (net 37 "COL2") (pinfunction "1") (pintype "passive"))
-    (pad "1" smd rect locked (at -3.275 -5.95 180) (size 2.6 2.6) (layers "B.Cu" "B.Paste" "B.Mask")
+    (pad "1" smd rect (at -3.275 -5.95 180) (size 2.6 2.6) (layers "B.Cu" "B.Paste" "B.Mask")
       (net 37 "COL2") (pinfunction "1") (pintype "passive"))
-    (pad "1" smd rect locked (at 3.275 -5.95 180) (size 2.6 2.6) (layers "F.Cu" "F.Paste" "F.Mask")
+    (pad "1" smd rect (at 3.275 -5.95 180) (size 2.6 2.6) (layers "F.Cu" "F.Paste" "F.Mask")
       (net 37 "COL2") (pinfunction "1") (pintype "passive"))
-    (pad "2" smd rect locked (at -8.275 -3.75 180) (size 2.6 2.6) (layers "F.Cu" "F.Paste" "F.Mask")
+    (pad "2" smd rect (at -8.275 -3.75 180) (size 2.6 2.6) (layers "F.Cu" "F.Paste" "F.Mask")
       (net 18 "Net-(D12-Pad2)") (pinfunction "2") (pintype "passive"))
-    (pad "2" thru_hole circle locked (at -5 3.8 180) (size 2.032 2.032) (drill 1.27) (layers *.Cu *.Mask)
+    (pad "2" thru_hole circle (at -5 3.8 180) (size 2.032 2.032) (drill 1.27) (layers *.Cu *.Mask)
       (net 18 "Net-(D12-Pad2)") (pinfunction "2") (pintype "passive"))
-    (pad "2" thru_hole circle locked (at 5 3.8 180) (size 2.032 2.032) (drill 1.27) (layers *.Cu *.Mask)
+    (pad "2" thru_hole circle (at 5 3.8 180) (size 2.032 2.032) (drill 1.27) (layers *.Cu *.Mask)
       (net 18 "Net-(D12-Pad2)") (pinfunction "2") (pintype "passive"))
-    (pad "2" smd rect locked (at 8.275 -3.75 180) (size 2.6 2.6) (layers "B.Cu" "B.Paste" "B.Mask")
+    (pad "2" smd rect (at 8.275 -3.75 180) (size 2.6 2.6) (layers "B.Cu" "B.Paste" "B.Mask")
       (net 18 "Net-(D12-Pad2)") (pinfunction "2") (pintype "passive"))
   )
@@
   (gr_line (start 86.7 77.15) (end 86.7 71.55) (layer "Edge.Cuts") (width 0.05))
   (gr_arc (start 193.763961 84.41) (mid 195.165494 86.24) (end 193.763961 88.07) (layer "Edge.Cuts") (width 0.05))
+  (gr_text "4" (at 137.26 61.55) (layer "B.SilkS")
+    (effects (font (size 1 1) (thickness 0.15)) (justify mirror))
+  )
   (gr_text "R3" (at 129.95 99.15) (layer "B.SilkS")
     (effects (font (size 1 1) (thickness 0.15)) (justify mirror))
@@
     (effects (font (size 1 1) (thickness 0.15)) (justify mirror))
   )
+  (gr_text "2" (at 141.1 56.64) (layer "B.SilkS")
+    (effects (font (size 1 1) (thickness 0.15)) (justify mirror))
+  )
   (gr_text "C1" (at 128.01 96) (layer "B.SilkS")
     (effects (font (size 1 1) (thickness 0.15)) (justify mirror))
   )
+  (gr_text "1" (at 137.3 53.85) (layer "B.SilkS")
+    (effects (font (size 1 1) (thickness 0.15)) (justify mirror))
+  )
   (gr_text "R5" (at 131.94 102.42) (layer "B.SilkS")
     (effects (font (size 1 1) (thickness 0.15)) (justify mirror))
   )
+  (gr_text "3" (at 141.12 59.23) (layer "B.SilkS")
+    (effects (font (size 1 1) (thickness 0.15)) (justify mirror))
+  )
   (gr_text "S6" (at 130.32 62.64) (layer "F.SilkS")
     (effects (font (size 1 1) (thickness 0.15)))
   )
+  (gr_text "4" (at 137.37 53.88) (layer "F.SilkS")
+    (effects (font (size 1 1) (thickness 0.15)))
+  )
+  (gr_text "3" (at 152.71 89.68) (layer "F.SilkS")
+    (effects (font (size 1 1) (thickness 0.15)))
+  )
+  (gr_text "RST" (at 134.26 97.3 90) (layer "F.SilkS")
+    (effects (font (size 0.6 0.6) (thickness 0.1)))
+  )
+  (gr_text "4" (at 155.2 89.63) (layer "F.SilkS")
+    (effects (font (size 1 1) (thickness 0.15)))
+  )
+  (gr_text "1" (at 147.89 89.69) (layer "F.SilkS")
+    (effects (font (size 1 1) (thickness 0.15)))
+  )
+  (gr_text "2" (at 150.28 89.7) (layer "F.SilkS")
+    (effects (font (size 1 1) (thickness 0.15)))
+  )
+  (gr_text "2" (at 141.17 59.18) (layer "F.SilkS")
+    (effects (font (size 1 1) (thickness 0.15)))
+  )
+  (gr_text "1" (at 137.33 61.58) (layer "F.SilkS")
+    (effects (font (size 1 1) (thickness 0.15)))
+  )
+  (gr_text "VCC" (at 134.28 104.44 90) (layer "F.SilkS")
+    (effects (font (size 0.6 0.6) (thickness 0.1)))
+  )
+  (gr_text "CLK" (at 134.29 99.9 90) (layer "F.SilkS")
+    (effects (font (size 0.6 0.6) (thickness 0.1)))
+  )
+  (gr_text "3" (at 141.17 56.64) (layer "F.SilkS")
+    (effects (font (size 1 1) (thickness 0.15)))
+  )
+  (gr_text "GND" (at 134.28 102.35 90) (layer "F.SilkS")
+    (effects (font (size 0.6 0.6) (thickness 0.1)))
+  )
+  (gr_text "DAT" (at 134.25 94.68 90) (layer "F.SilkS")
+    (effects (font (size 0.6 0.6) (thickness 0.1)))
+  )
   (segment (start 92.529674 56.924432) (end 98.435568 56.924432) (width 0.35) (layer "F.Cu") (net 2))

Commit message: started routing
Parts:
- moved R1 84.0 mm to (90.2, 97.4), turned to 180 degrees
- moved R2 81.1 mm to (94.6, 97.4)
Connections:
- U1 pad 14: COL2 -> ROW3
- U1 pad 17: ROW3 -> COL2
- U14 pad 14: COL2 -> ROW3
- U14 pad 17: ROW3 -> COL2
Routing:
- net ROW0: track 13.6 -> 131.3 mm, vias 1 -> 9
- net COL4: track 28.4 -> 130.6 mm, vias 1 -> 4
- net ROW1: track 14.5 -> 113.8 mm, vias 1 -> 5
- net COL5: track 24.5 -> 119.7 mm, vias 1 -> 4
- net COL3: track 28.8 -> 107.2 mm, vias 1 -> 4
- net ROW2: track 15.5 -> 92.0 mm, vias 1 -> 6
- net Net-(D13-Pad2): track 0.00 -> 57.5 mm, vias 0 -> 3
- net Net-(D15-Pad2): track 0.00 -> 54.7 mm, vias 0 -> 3
- net Net-(D14-Pad2): track 0.00 -> 54.2 mm, vias 0 -> 4
- net Net-(D9-Pad2): track 0.00 -> 52.4 mm, vias 0 -> 3
- net COL2: track 25.5 -> 72.9 mm, vias 1 -> 4
- net Net-(D16-Pad2): track 0.00 -> 42.6 mm
- net Net-(D17-Pad2): track 0.00 -> 41.4 mm, vias 0 -> 2
- net Net-(D18-Pad2): track 0.00 -> 40.2 mm, vias 0 -> 2
- net Net-(D19-Pad2): track 0.00 -> 36.3 mm
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