File: PCB/TPS42-Shield/TPS42-Shield.kicad_pcb (KiCad board)
At the start: 2 copper layers, 36.9 x 43.9 mm, 33 parts, among them J1 PJ-320A, J10 FH12-10S-0.5SH, J11 Conn_01x06, J12 Conn_01x01, J2 Conn_01x06, J3 OLED, J4 PJ-320A, J5 Conn_01x06, J6 OLED, J7 FH12-10S-0.5SH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

Commit message: make it reversable (I)
Parts:
- removed C4: 560pF/680pF, Capacitor_SMD:C_0603_1608Metric_Pad1.08x0.95mm_HandSolder
- removed C5, C6: 1uF, Capacitor_SMD:C_0603_1608Metric_Pad1.08x0.95mm_HandSolder
- removed FB3, FB4: Ferrite_Bead, Resistor_SMD:R_0805_2012Metric_Pad1.20x1.40mm_HandSolder
- removed J1: PJ-320A, TPS42-Shield:MJ-4PP-9
- removed J10: FH12-10S-0.5SH, Connector_FFC-FPC:Hirose_FH12-10S-0.5SH_1x10-1MP_P0.50mm_Horizontal
- removed J11, J2: Conn_01x06, Connector_PinHeader_2.54mm:PinHeader_2x03_P2.54mm_Vertical
- removed J12, J9: Conn_01x01, Connector_PinHeader_2.54mm:PinHeader_1x01_P2.54mm_Vertical
- removed J3: OLED, TPS42-Shield:OLED
- removed R2: 10kΩ, Resistor_SMD:R_0603_1608Metric_Pad0.98x0.95mm_HandSolder
- removed mouse-bite-2mm-slot (x7): VAL**, TPS42-Shield:mouse-bite-2mm-slot
- added H1: MouseBite, TPS42-Shield:mouse-bite-2mm-slot, F.Cu at (88.1, 39.6)
- added H2: MouseBite, TPS42-Shield:mouse-bite-2mm-slot, F.Cu at (85.3, 39.6)
- added JP10: Jumper_2_Open, Jumper:SolderJumper-2_P1.3mm_Open_TrianglePad1.0x1.5mm, F.Cu at (51.1, 29.6)
- added JP11: Jumper_2_Open, Jumper:SolderJumper-2_P1.3mm_Open_TrianglePad1.0x1.5mm, F.Cu at (42.5, 29.6)
- added JP12: Jumper_2_Open, Jumper:SolderJumper-2_P1.3mm_Open_TrianglePad1.0x1.5mm, F.Cu at (46.8, 29.6)
- added JP13: Jumper_2_Open, Jumper:SolderJumper-2_P1.3mm_Open_TrianglePad1.0x1.5mm, F.Cu at (55.5, 26.1)
- added JP14: Jumper_2_Open, Jumper:SolderJumper-2_P1.3mm_Open_TrianglePad1.0x1.5mm, F.Cu at (51.1, 33.2)
- added JP15: Jumper_2_Open, Jumper:SolderJumper-2_P1.3mm_Open_TrianglePad1.0x1.5mm, F.Cu at (51.1, 26.1)
- added JP16: Jumper_2_Open, Jumper:SolderJumper-2_P1.3mm_Open_TrianglePad1.0x1.5mm, F.Cu at (42.5, 33.2)
- added JP17: Jumper_2_Open, Jumper:SolderJumper-2_P1.3mm_Open_TrianglePad1.0x1.5mm, F.Cu at (46.8, 26.1)
- added JP18: Jumper_2_Open, Jumper:SolderJumper-2_P1.3mm_Open_TrianglePad1.0x1.5mm, F.Cu at (42.5, 26.1)
- added JP3: Jumper_2_Open, Jumper:SolderJumper-2_P1.3mm_Open_TrianglePad1.0x1.5mm, F.Cu at (92.9, 49.0)
- added JP4: Jumper_2_Open, Jumper:SolderJumper-2_P1.3mm_Open_TrianglePad1.0x1.5mm, F.Cu at (92.9, 51.7)
- added JP5: Jumper_2_Open, Jumper:SolderJumper-2_P1.3mm_Open_TrianglePad1.0x1.5mm, B.Cu at (98.3, 51.7)
- added JP6: Jumper_2_Open, Jumper:SolderJumper-2_P1.3mm_Open_TrianglePad1.0x1.5mm, B.Cu at (98.3, 49.0)
- added JP7: Jumper_2_Open, Jumper:SolderJumper-2_P1.3mm_Open_TrianglePad1.0x1.5mm, B.Cu at (92.9, 49.0)
- added JP8: Jumper_2_Open, Jumper:SolderJumper-2_P1.3mm_Open_TrianglePad1.0x1.5mm, B.Cu at (92.9, 51.7)
- added JP9: Jumper_2_Open, Jumper:SolderJumper-2_P1.3mm_Open_TrianglePad1.0x1.5mm, F.Cu at (46.8, 33.2)
- J4: footprint TPS42-Shield:MJ-4PP-9 -> TPS42-Shield:MJ-4PP-9-reversable
- J8: moved to F.Cu
- JP1, JP2: value Jumper_3_Open -> Jumper_2_Open; footprint Jumper:SolderJumper-3_P2.0mm_Open_TrianglePad1.0x1.5mm -> Jumper:SolderJumper-2_P1.3mm_Open_TrianglePad1.0x1.5mm
- moved JP2 63.7 mm to (98.3, 49.0)
- moved C1 50.2 mm to (102.7, 53.2), turned to 180 degrees
- moved J8 48.6 mm to (98.3, 56.3)
- moved JP1 46.8 mm to (98.3, 51.7)
- moved FB1 46.2 mm to (103.6, 46.1), turned to -90 degrees
- moved R1 45.4 mm to (102.7, 50.0), turned to 180 degrees
- moved C3 44.8 mm to (102.7, 51.6), turned to 180 degrees
- moved J7 43.7 mm to (95.8, 39.2)
- moved J6 42.9 mm to (77.6, 44.8), turned to 0 degrees
- moved J4 39.5 mm to (68.2, 51.1)
- moved FB2 38.8 mm to (87.9, 46.1)
- moved C2 35.7 mm to (87.9, 49.9), turned to 90 degrees
- moved J5 33.6 mm to (75.0, 56.3), turned to -90 degrees
Connections:
- C1 pad 1: /L_DISP -> +3V3
- J4 pad 1: Net-(J4-Pad1) -> VCC
- J4 pad 4: Net-(J4-Pad4) -> GND
- J5 pad 1: Net-(J5-Pad1) -> unconnected-(J5-Pad1)
- J5 pad 2: Net-(J4-Pad4) -> GND
- J5 pad 3: Net-(J5-Pad3) -> unconnected-(J5-Pad3)
- J5 pad 4: Net-(J4-Pad2) -> Net-(J5-Pad4)
- J5 pad 5: Net-(J4-Pad1) -> VCC
- J5 pad 6: unconnected-(J5-Pad6) -> Net-(J5-Pad6)
- J6 pad 1: Net-(J5-Pad1) -> Net-(J6-Pad1)
- J6 pad 2: Net-(J5-Pad3) -> Net-(J6-Pad2)
- J6 pad 3: Net-(J4-Pad1) -> Net-(J6-Pad3)
- J6 pad 4: Net-(J4-Pad4) -> Net-(J6-Pad4)
- J7 pad 5: /L_DISP -> +3V3
- J8 pad 1: /L_DAT -> Net-(J8-Pad1)
- J8 pad 3: /L_CLK -> Net-(J8-Pad3)
- J8 pad 4: /L_EIN -> Net-(J8-Pad4)
- J8 pad 6: /L_CS -> Net-(J8-Pad6)
- JP1 pad 1: Net-(J9-Pad1) -> Net-(J8-Pad6)
- JP1 pad 2: /L_DISP -> /L_CS
- JP2 pad 1: Net-(J12-Pad1) -> Net-(J8-Pad4)
- JP2 pad 2: /R_DISP -> /L_EIN
Routing:
- net GNDA: track 62.3 -> 15.3 mm, vias 8 -> 1
- net +3V3: track 87.8 -> 48.9 mm, vias 5 -> 6
- net /R_CS: track 36.5 -> 0.00 mm, vias 2 -> 0
- net /L_DISP: track 34.2 -> 0.00 mm, vias 1 -> 0
- net /R_CLK: track 32.7 -> 0.00 mm, vias 2 -> 0
- net /R_DISP: track 32.4 -> 0.00 mm, vias 1 -> 0
- net VDDA: track 61.6 -> 31.1 mm, vias 2 -> 4
- net /R_EIN: track 29.9 -> 0.00 mm, vias 1 -> 0
- net /R_DAT: track 26.2 -> 0.00 mm, vias 2 -> 0
- net Net-(J2-Pad1): track 19.1 -> 0.00 mm, vias 1 -> 0
- net Net-(J1-Pad2): track 19.0 -> 0.00 mm
- net Net-(J4-Pad4): track 17.5 -> 0.00 mm, vias 1 -> 0
- net Net-(J4-Pad1): track 17.4 -> 0.00 mm, vias 1 -> 0
- net /L_EIN: track 41.7 -> 24.8 mm, vias 1 -> 3
- net Net-(J12-Pad1): track 15.6 -> 0.00 mm, vias 3 -> 0
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Other:
- board size 36.9 x 43.9 mm -> 35.9 x 25.8 mm
- board text removed: "LEFT"
- board text removed: "RIGHT"
