File: PCB/TPS42-Serial-OLED-Shield/TPS42-Serial-OLED-Shield.kicad_pcb (KiCad board)
At the start: 2 copper layers, 17.7 x 25.8 mm, 13 parts, among them J4 PJ-320A, J5 Conn_01x06, J6 OLED

Commit message: renaming
Parts:
- J4: footprint TPS42-Shield:MJ-4PP-9-reversable -> TPS42-Serial-OLED-Shield:MJ-4PP-9-reversable
- J6: footprint TPS42-Shield:OLED -> TPS42-Serial-OLED-Shield:OLED
Changed lines of the file:
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@@
   (net 11 "Net-(J6-Pad2)")
   (net 12 "Net-(J6-Pad1)")
-  (footprint "TPS42-Shield:OLED" (layer "F.Cu")
+  (footprint "TPS42-Serial-OLED-Shield:OLED" (layer "F.Cu")
     (at 77.561543 44.778457)
     (descr "Connecteur 6 pins")
     (tags "CONN DEV")
-    (property "Sheetfile" "TPS42-Shield.kicad_sch")
+    (property "Sheetfile" "TPS42-Serial-OLED-Shield.kicad_sch")
     (property "Sheetname" "")
     (attr through_hole)
@@
     (descr "SMD Solder Jumper, 1x1.5mm Triangular Pads, 0.3mm gap, open")
     (tags "solder jumper open")
-    (property "Sheetfile" "TPS42-Shield.kicad_sch")
+    (property "Sheetfile" "TPS42-Serial-OLED-Shield.kicad_sch")
     (property "Sheetname" "")
     (attr exclude_from_pos_files)
@@
     (descr "SMD Solder Jumper, 1x1.5mm Triangular Pads, 0.3mm gap, open")
     (tags "solder jumper open")
-    (property "Sheetfile" "TPS42-Shield.kicad_sch")
+    (property "Sheetfile" "TPS42-Serial-OLED-Shield.kicad_sch")
     (property "Sheetname" "")
     (attr exclude_from_pos_files)
@@
     (descr "SMD Solder Jumper, 1x1.5mm Triangular Pads, 0.3mm gap, open")
     (tags "solder jumper open")
-    (property "Sheetfile" "TPS42-Shield.kicad_sch")
+    (property "Sheetfile" "TPS42-Serial-OLED-Shield.kicad_sch")
     (property "Sheetname" "")
     (attr exclude_from_pos_files)
@@
     (descr "SMD Solder Jumper, 1x1.5mm Triangular Pads, 0.3mm gap, open")
     (tags "solder jumper open")
-    (property "Sheetfile" "TPS42-Shield.kicad_sch")
+    (property "Sheetfile" "TPS42-Serial-OLED-Shield.kicad_sch")
     (property "Sheetname" "")
     (attr exclude_from_pos_files)
@@
     (descr "SMD Solder Jumper, 1x1.5mm Triangular Pads, 0.3mm gap, open")
     (tags "solder jumper open")
-    (property "Sheetfile" "TPS42-Shield.kicad_sch")
+    (property "Sheetfile" "TPS42-Serial-OLED-Shield.kicad_sch")
     (property "Sheetname" "")
     (attr exclude_from_pos_files)
@@
     (descr "SMD Solder Jumper, 1x1.5mm Triangular Pads, 0.3mm gap, open")
     (tags "solder jumper open")
-    (property "Sheetfile" "TPS42-Shield.kicad_sch")
+    (property "Sheetfile" "TPS42-Serial-OLED-Shield.kicad_sch")
     (property "Sheetname" "")
     (attr exclude_from_pos_files)
@@
       ))
   )
-  (footprint "TPS42-Shield:MJ-4PP-9-reversable" (layer "B.Cu")
+  (footprint "TPS42-Serial-OLED-Shield:MJ-4PP-9-reversable" (layer "B.Cu")
     (at 68.161543 51.063457 -90)
-    (property "Sheetfile" "TPS42-Shield.kicad_sch")
+    (property "Sheetfile" "TPS42-Serial-OLED-Shield.kicad_sch")
     (property "Sheetname" "")
     (attr through_hole)
@@
     (descr "Through hole straight pin header, 2x03, 2.54mm pitch, double rows")
     (tags "Through hole pin header THT 2x03 2.54mm double row")
-    (property "Sheetfile" "TPS42-Shield.kicad_sch")
+    (property "Sheetfile" "TPS42-Serial-OLED-Shield.kicad_sch")
     (property "Sheetname" "")
     (attr through_hole)
@@
     (descr "SMD Solder Jumper, 1x1.5mm Triangular Pads, 0.3mm gap, open")
     (tags "solder jumper open")
-    (property "Sheetfile" "TPS42-Shield.kicad_sch")
+    (property "Sheetfile" "TPS42-Serial-OLED-Shield.kicad_sch")
     (property "Sheetname" "")
     (attr exclude_from_pos_files)
@@
     (descr "SMD Solder Jumper, 1x1.5mm Triangular Pads, 0.3mm gap, open")
     (tags "solder jumper open")
-    (property "Sheetfile" "TPS42-Shield.kicad_sch")
+    (property "Sheetfile" "TPS42-Serial-OLED-Shield.kicad_sch")
     (property "Sheetname" "")
     (attr exclude_from_pos_files)
@@
     (descr "SMD Solder Jumper, 1x1.5mm Triangular Pads, 0.3mm gap, open")
     (tags "solder jumper open")
-    (property "Sheetfile" "TPS42-Shield.kicad_sch")
+    (property "Sheetfile" "TPS42-Serial-OLED-Shield.kicad_sch")
     (property "Sheetname" "")
     (attr exclude_from_pos_files)
@@
     (descr "SMD Solder Jumper, 1x1.5mm Triangular Pads, 0.3mm gap, open")
     (tags "solder jumper open")
-    (property "Sheetfile" "TPS42-Shield.kicad_sch")
-    (property "Sheetname" "")
-    (attr exclude_from_pos_files)
+    (property "Sheetfile" "TPS42-Serial-OLED-Shield.kicad_sch")
+    (property "Sheetname" "")
+    (attr exclude_from_pos_files)

Commit message: finalizing
Parts:
- JP13: moved to B.Cu
- JP14: moved to F.Cu
- moved JP13 12.8 mm to (85.0, 48.9)
- moved JP14 12.8 mm to (85.0, 48.9)
Routing:
- net Net-(J4-Pad2): track 12.7 -> 21.5 mm, vias 0 -> 1
- net Net-(J5-Pad4): track 11.3 -> 15.0 mm, vias 1 -> 0
- net Net-(J5-Pad6): track 13.8 -> 11.5 mm, vias 0 -> 1
- net /SDA: track 36.5 -> 35.9 mm
Other:
- board text added: "${Revision}"
- board text added: "Left"

Commit message: removed serial jumber
Parts:
- removed JP13, JP14: Jumper_2_Open, Jumper:SolderJumper-2_P1.3mm_Open_TrianglePad1.0x1.5mm
Connections:
- J5 pad 4: Net-(J5-Pad4) -> unconnected-(J5-Pad4)
- J5 pad 6: Net-(J5-Pad6) -> Net-(J4-Pad2)
Routing:
- net Net-(J5-Pad4): track 15.0 -> 0.00 mm
- net Net-(J5-Pad6): track 11.5 -> 0.00 mm, vias 1 -> 0
- net unconnected-(J5-Pad4): track 0.00 -> 7.92 mm
- net Net-(J4-Pad2): track 21.5 -> 20.4 mm, vias 1 -> 0
